Commit message: URDF with angles

File: Project/urdf/opendog.urdf (robot description, URDF)
Before this commit: robot opendog, 13 links, 12 joints
Joints:
- joint coude_ar_d: limit effort=1 velocity=20 -> lower=-0.872665 upper=0.698132 effort=1 velocity=20; origin xyz=0.0279938 1.83141e-07 0.095 rpy=-2.65094e-24 -1.5708 0 -> xyz=0.0319278 -1.83141e-07 0.1815 rpy=3.14159 1.5708 0
- joint coude_ar_g: limit effort=1 velocity=20 -> lower=-0.349066 upper=0.872665 effort=1 velocity=20; origin xyz=0.0319278 1.83141e-07 0.1995 rpy=1.38778e-15 -1.5708 0 -> xyz=0.0319278 -1.83141e-07 0.077 rpy=-3.14159 1.5708 0
- joint coude_avt_d: limit effort=1 velocity=20 -> lower=-0.349066 upper=0.872665 effort=1 velocity=20
- joint coude_avt_g: limit effort=1 velocity=20 -> lower=-0.872665 upper=0.698132 effort=1 velocity=20; origin xyz=0.0279938 -1.83141e-07 -0.093 rpy=-3.14159 1.5708 0 -> xyz=0.0319938 -1.83141e-07 -0.095 rpy=-3.14159 1.5708 0
- joint epaule_ar_d: limit effort=1 velocity=20 -> lower=-0.523599 upper=1.39626 effort=1 velocity=20; origin xyz=-0.126016 0.359695 0.0733429 rpy=-1.5708 6.69971e-24 -3.14159 -> xyz=-0.126016 0.0833899 0.0733429 rpy=1.5708 -4.75723e-14 -3.14159
- joint epaule_ar_g: limit effort=1 velocity=20 -> lower=-0.523599 upper=1.39626 effort=1 velocity=20; origin xyz=0.123746 0.0650189 0.0733429 rpy=-1.5708 -3.66374e-15 6.38027e-10 -> xyz=0.123746 0.341324 0.0733429 rpy=1.5708 -1.19349e-15 6.38026e-10
- joint epaule_avt_d: limit effort=1 velocity=20 -> lower=-0.523599 upper=1.39626 effort=1 velocity=20; origin xyz=-0.126016 -0.0654131 0.0733429 rpy=1.5708 1.33279e-23 -3.14159 -> xyz=-0.126016 -0.0654131 0.0733429 rpy=1.5708 2.03529e-14 -3.14159
- joint epaule_avt_g: limit effort=1 velocity=20 -> lower=-0.523599 upper=1.39626 effort=1 velocity=20; origin xyz=0.123746 -0.360089 0.0733429 rpy=1.5708 4.49058e-09 6.38027e-10 -> xyz=0.123746 -0.360089 0.0733429 rpy=1.5708 -4.4944e-14 6.38027e-10
- joint poignet_ar_d: limit effort=1 velocity=20 -> lower=-2.35619 upper=2.35619 effort=1 velocity=20; origin xyz=-4.16334e-15 0.2 -0.065516 rpy=1.22677e-16 4.26771e-14 -3.98097e-09 -> xyz=-4.05231e-15 0.2 -0.065516 rpy=3.14159 -4.48145e-15 -9.21485e-15
- joint poignet_ar_g: limit effort=1 velocity=20 -> lower=-2.35619 upper=2.35619 effort=1 velocity=20; origin xyz=-4.21885e-15 0.2 -0.065516 rpy=1.08117e-14 8.49257e-14 8.32667e-16 -> xyz=-4.32987e-15 0.2 -0.065516 rpy=-3.14159 -9.28741e-16 -3.33067e-16
- joint poignet_avt_d: limit effort=1 velocity=20 -> lower=-2.35619 upper=2.35619 effort=1 velocity=20; origin xyz=-4.16334e-15 0.2 -0.065516 rpy=1.22677e-16 1.01389e-13 -3.98097e-09 -> xyz=-4.21885e-15 0.2 -0.065516 rpy=-3.14159 8.47616e-16 3.33067e-16
- joint poignet_avt_g: limit effort=1 velocity=20 -> lower=-2.35619 upper=2.35619 effort=1 velocity=20; origin xyz=-4.21885e-15 0.2 -0.065516 rpy=-1.25065e-14 4.26771e-14 -3.98097e-09 -> xyz=-4.27436e-15 0.2 -0.065516 rpy=-3.14159 -4.05626e-17 -2.77556e-16
