Commit message: URDF avec frames pour les pieds

File: Project/urdf/robot.urdf (robot description, URDF)
Before this commit: robot opendog, 13 links, 12 joints
Links:
- removed link avantbras
- removed link avantbras_2
- removed link avantbras_3
- removed link avantbras_4
- removed link bras
- removed link bras_2
- removed link bras_3
- removed link bras_4
- removed link chassis
- removed link epaule
- removed link epaule_2
- removed link epaulemiroir
- removed link epaulemiroir_2
- added link body, mass 6.64; collision mesh filename=package://body_1.stl; collision mesh filename=package://body_10.stl
- added link foot_bl, mass 1e-9
- added link foot_br, mass 1e-9
- added link foot_fl, mass 1e-9
- added link foot_lr, mass 1e-9
- added link hip, mass 1.23; collision mesh filename=package://ams_3.stl; collision mesh filename=package://ams_4.stl
- added link hip_2, mass 1.23; collision mesh filename=package://ams_3.stl; collision mesh filename=package://ams_4.stl
- added link lowerleg, mass 0.34; collision mesh filename=package://foot.stl; collision mesh filename=package://lowerleg_1.stl
- added link lowerleg_2, mass 0.34; collision mesh filename=package://foot.stl; collision mesh filename=package://lowerleg_1.stl
- added link lowerleg_3, mass 0.34; collision mesh filename=package://foot.stl; collision mesh filename=package://lowerleg_1.stl
- added link lowerleg_4, mass 0.34; collision mesh filename=package://foot.stl; collision mesh filename=package://lowerleg_1.stl
- added link mirrorhip, mass 1.23081; collision mesh filename=package://ams_5.stl; collision mesh filename=package://ams_6.stl
- added link mirrorhip_2, mass 1.23081; collision mesh filename=package://ams_5.stl; collision mesh filename=package://ams_6.stl
- added link upperleg, mass 0.97; collision mesh filename=package://ams_1.stl; collision mesh filename=package://ams_2.stl
- added link upperleg_2, mass 0.97; collision mesh filename=package://ams_1.stl; collision mesh filename=package://ams_2.stl
- added link upperleg_3, mass 0.97; collision mesh filename=package://ams_1.stl; collision mesh filename=package://ams_2.stl
- added link upperleg_4, mass 0.97; collision mesh filename=package://ams_1.stl; collision mesh filename=package://ams_2.stl
Joints:
- removed joint coude_ar_d
- removed joint coude_ar_g
- removed joint coude_avt_d
- removed joint coude_avt_g
- removed joint epaule_ar_d
- removed joint epaule_ar_g
- removed joint epaule_avt_d
- removed joint epaule_avt_g
- removed joint poignet_ar_d
- removed joint poignet_ar_g
- removed joint poignet_avt_d
- removed joint poignet_avt_g
- added joint ankle_bl: type revolute, parent upperleg_3, child lowerleg_3, origin xyz=-4.32987e-15 0.2 -0.065516 rpy=-3.14159 -9.28741e-16 -3.33067e-16, axis 0 0 1, limit lower=-2.35619 upper=2.35619 effort=1 velocity=20
- added joint ankle_br: type revolute, parent upperleg_4, child lowerleg_4, origin xyz=-4.05231e-15 0.2 -0.065516 rpy=3.14159 -4.48145e-15 -9.21485e-15, axis 0 0 1, limit lower=-2.35619 upper=2.35619 effort=1 velocity=20
- added joint ankle_fl: type revolute, parent upperleg, child lowerleg, origin xyz=-4.27436e-15 0.2 -0.065516 rpy=-3.14159 -4.05626e-17 -2.77556e-16, axis 0 0 1, limit lower=-2.35619 upper=2.35619 effort=1 velocity=20
- added joint ankle_fr: type revolute, parent upperleg_2, child lowerleg_2, origin xyz=-4.21885e-15 0.2 -0.065516 rpy=-3.14159 8.47616e-16 3.33067e-16, axis 0 0 1, limit lower=-2.35619 upper=2.35619 effort=1 velocity=20
- added joint foot_bl_frame: type fixed, parent lowerleg_3, child foot_bl, origin xyz=1.44661e-05 -0.195916 -0.0978296 rpy=-1.5708 -1.5708 0, axis 0 0 0
- added joint foot_br_frame: type fixed, parent lowerleg_4, child foot_br, origin xyz=1.44661e-05 -0.195916 -0.0978296 rpy=-1.5708 1.5708 0, axis 0 0 0
- added joint foot_fl_frame: type fixed, parent lowerleg, child foot_fl, origin xyz=1.44661e-05 -0.195916 -0.0978296 rpy=-1.5708 -1.5708 0, axis 0 0 0
- added joint foot_lr_frame: type fixed, parent lowerleg_2, child foot_lr, origin xyz=1.44661e-05 -0.195916 -0.0978296 rpy=-1.5708 1.5708 0, axis 0 0 0
- added joint hip_bl: type revolute, parent body, child mirrorhip_2, origin xyz=0.123746 0.341324 0.0733429 rpy=1.5708 -1.19349e-15 6.38026e-10, axis 0 0 1, limit lower=-0.523599 upper=1.39626 effort=1 velocity=20
- added joint hip_br: type revolute, parent body, child hip_2, origin xyz=-0.126016 0.0833899 0.0733429 rpy=1.5708 -4.75723e-14 -3.14159, axis 0 0 1, limit lower=-0.523599 upper=1.39626 effort=1 velocity=20
- added joint hip_fl: type revolute, parent body, child hip, origin xyz=0.123746 -0.360089 0.0733429 rpy=1.5708 -4.4944e-14 6.38027e-10, axis 0 0 1, limit lower=-0.523599 upper=1.39626 effort=1 velocity=20
- added joint hip_fr: type revolute, parent body, child mirrorhip, origin xyz=-0.126016 -0.0654131 0.0733429 rpy=1.5708 2.03529e-14 -3.14159, axis 0 0 1, limit lower=-0.523599 upper=1.39626 effort=1 velocity=20
- added joint knee_bl: type revolute, parent mirrorhip_2, child upperleg_3, origin xyz=0.0319278 -1.83141e-07 0.077 rpy=-3.14159 1.5708 0, axis 0 0 1, limit lower=-0.349066 upper=0.872665 effort=1 velocity=20
- added joint knee_br: type revolute, parent hip_2, child upperleg_4, origin xyz=0.0319278 -1.83141e-07 0.1815 rpy=3.14159 1.5708 0, axis 0 0 1, limit lower=-0.872665 upper=0.698132 effort=1 velocity=20
- added joint knee_fl: type revolute, parent hip, child upperleg, origin xyz=0.0319938 -1.83141e-07 -0.095 rpy=-3.14159 1.5708 0, axis 0 0 1, limit lower=-0.872665 upper=0.698132 effort=1 velocity=20
- added joint knee_fr: type revolute, parent mirrorhip, child upperleg_2, origin xyz=0.0319278 -1.83141e-07 -0.1995 rpy=-3.14159 1.5708 0, axis 0 0 1, limit lower=-0.349066 upper=0.872665 effort=1 velocity=20

Commit message: URDF avec frame centrale

File: Project/urdf/robot.urdf (robot description, URDF)
Before this commit: robot opendog, 17 links, 16 joints
Links:
- added link center, mass 1e-9
- link lowerleg: geometry collision mesh filename=package://lowerleg_1.stl; collision mesh filename=package://lowerleg_2.stl
- link lowerleg_2: geometry collision mesh filename=package://lowerleg_1.stl; collision mesh filename=package://lowerleg_2.stl
- link lowerleg_3: geometry collision mesh filename=package://lowerleg_1.stl; collision mesh filename=package://lowerleg_2.stl
- link lowerleg_4: geometry collision mesh filename=package://lowerleg_1.stl; collision mesh filename=package://lowerleg_2.stl
Joints:
- added joint center_frame: type fixed, parent body, child center, origin xyz=-0.00114401 -0.00271308 0.0708426 rpy=1.07093e-25 3.41171e-16 -1.5708, axis 0 0 0

Commit message: new urdf

File: Project/urdf/robot.urdf (robot description, URDF)
Before this commit: robot opendog, 18 links, 17 joints
Links:
- removed link foot_lr
- added link foot_fr, mass 1e-9
Joints:
- removed joint foot_lr_frame
- added joint foot_fr_frame: type fixed, parent lowerleg_2, child foot_fr, origin xyz=1.44661e-05 -0.195916 -0.0978296 rpy=-1.5708 1.5708 0, axis 0 0 0
